Commit message: feat: manipulator control interface

File: uuv_description/urdf/bluerov2_description.urdf.xacro (robot description, xacro)
@@ -24,5 +24,5 @@
         </collision>
     </link>
-    <!-- ============================= MANIPULATOR 1.4124 kg ===================================
+    <!-- ============================= MANIPULATOR 1.4124 kg =================================== -->
     <link name="manipulator_base_footprint" />
     <joint name="manipulator_base_footprint_joint" type="fixed">
@@ -35,4 +35,4 @@
       description_package="uuv_description">
       <origin xyz="0 0 0" rpy="0 0 0" />
-    </xacro:alpha_urdf> -->
+    </xacro:alpha_urdf>
 </robot>

File: uuv_description/urdf/manipulator/end_effectors/standard_jaws.urdf.xacro (robot description, xacro)
@@ -116,4 +116,13 @@
       <mimic joint="${axis_a}" multiplier="51" offset="0" />
     </joint>
+    <transmission name="transmission_rs1_130_joint">
+      <type>transmission_interface/SimpleTransmission</type>
+      <joint name="${prefix}rs1_130_joint">
+        <hardwareInterface>hardware_interface/EffortJointInterface</hardwareInterface>
+      </joint>
+      <actuator name="rs1_130_joint_motor">
+        <mechanicalReduction>1</mechanicalReduction>
+      </actuator>
+    </transmission>
     <joint name="${prefix}rs1_139_joint" type="revolute">
       <origin xyz="0 -0.0155 0.0069" rpy="0 0 0" />
@@ -124,4 +133,13 @@
       <mimic joint="${prefix}rs1_130_joint" multiplier="1" offset="0" />
     </joint>
+    <transmission name="transmission_rs1_139_joint">
+      <type>transmission_interface/SimpleTransmission</type>
+      <joint name="${prefix}rs1_139_joint">
+        <hardwareInterface>hardware_interface/EffortJointInterface</hardwareInterface>
+      </joint>
+      <actuator name="rs1_139_joint_motor">
+        <mechanicalReduction>1</mechanicalReduction>
+      </actuator>
+    </transmission>
     <joint name="${prefix}tool_joint" type="fixed">
       <origin xyz="0 0 0.04" rpy="0 -1.571 0" />

File: uuv_description/urdf/manipulator/manipulator.urdf.xacro (robot description, xacro)
@@ -210,4 +210,9 @@
       </inertial>
     </link>
+    <gazebo>
+      <plugin name="gazebo_ros_control" filename="libgazebo_ros_control.so">
+        <robotNamespace>/manipulator</robotNamespace>
+      </plugin>
+    </gazebo>
     <joint name="${prefix}base_joint" type="fixed">
       <xacro:insert_block name="origin" />
@@ -227,4 +232,13 @@
       <limit effort="9.0" lower="0.0" upper="6.10" velocity="0.5" />
     </joint>
+    <transmission name="transmission_axis_e">
+      <type>transmission_interface/SimpleTransmission</type>
+      <joint name="${prefix}axis_e">
+        <hardwareInterface>hardware_interface/EffortJointInterface</hardwareInterface>
+      </joint>
+      <actuator name="axis_e_motor">
+        <mechanicalReduction>1</mechanicalReduction>
+      </actuator>
+    </transmission>
     <joint name="${prefix}axis_d" type="revolute">
       <parent link="${prefix}m2_1_1_link" />
@@ -235,4 +249,13 @@
       <limit effort="9.0" lower="-3.49" upper="3.49" velocity="0.5" />
     </joint>
+    <transmission name="transmission_axis_d">
+      <type>transmission_interface/SimpleTransmission</type>
+      <joint name="${prefix}axis_d">
+        <hardwareInterface>hardware_interface/EffortJointInterface</hardwareInterface>
+      </joint>
+      <actuator name="axis_d_motor">
+        <mechanicalReduction>1</mechanicalReduction>
+      </actuator>
+    </transmission>
     <joint name="${prefix}axis_c" type="revolute">
       <parent link="${prefix}m2_joint_link" />
@@ -242,4 +265,13 @@
       <limit effort="9.0" lower="0.0" upper="3.22" velocity="0.5" />
     </joint>
+    <transmission name="transmission_axis_c">
+      <type>transmission_interface/SimpleTransmission</type>
+      <joint name="${prefix}axis_c">
+        <hardwareInterface>hardware_interface/EffortJointInterface</hardwareInterface>
+      </joint>
+      <actuator name="axis_c_motor">
+        <mechanicalReduction>1</mechanicalReduction>
+      </actuator>
+    </transmission>
     <joint name="${prefix}axis_b" type="revolute">
       <parent link="${prefix}m2_1_2_link" />
@@ -249,4 +281,13 @@
       <limit effort="9.0" lower="0.0" upper="3.22" velocity="0.5" />
     </joint>
+    <transmission name="transmission_axis_b">
+      <type>transmission_interface/SimpleTransmission</type>
+      <joint name="${prefix}axis_b">
+        <hardwareInterface>hardware_interface/EffortJointInterface</hardwareInterface>
+      </joint>
+      <actuator name="axis_b_motor">
+        <mechanicalReduction>1</mechanicalReduction>
+      </actuator>
+    </transmission>
     <joint name="${prefix}ee_joint" type="fixed">
       <origin rpy="0 0 0" xyz="0 0 0.09975" />
